File: Extras/ScottoModules/ScottoModules.kicad_pcb (KiCad board)
At the start: 2 copper layers, 57.2 x 57.1 mm, 27 parts, among them J1 USB_C, SW1 SW_Push, U1 STM32F072CBT6, U3 XC6206, U4 USBLC6-2SC6

Commit message: Fix JLCPCB Rotation
Parts:
- C6: value 10uf -> 10uF
- C7: value 100nf -> 100nF
Connections:
- S4 pad 1: (no net) -> Net-(S1-Pad1) (x2)
- S4 pad 2: (no net) -> Net-(D4-A) (x2)
- S6 pad 1: (no net) -> Net-(S3-Pad1)
- S6 pad 2: (no net) -> Net-(D6-A)
Changed lines of the file:
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@@
 		(pad_to_mask_clearance 0)
 		(allow_soldermask_bridges_in_footprints no)
-		(grid_origin 430.267448 34.035023)
+		(grid_origin 436.729948 55.707522)
 		(pcbplotparams
 			(layerselection 0x00010fc_ffffffff)
@@
 			)
 		)
+		(property ki_fp_filters "R_*")
+		(sheetname "Root")
+		(sheetfile "ScottoModules.kicad_sch")
 		(attr smd)
 		(fp_line
@@
 			)
 		)
-		(property "Value" "10uf"
+		(property "Value" "10uF"
 			(at 0.000001 -1.430002 180)
 			(layer "B.Fab")
@@
 			)
 		)
+		(property ki_fp_filters "C_*")
+		(sheetname "Root")
+		(sheetfile "ScottoModules.kicad_sch")
 		(attr smd)
 		(fp_line
@@
 			)
 		)
+		(property ki_fp_filters "C_*")
+		(sheetname "Root")
+		(sheetfile "ScottoModules.kicad_sch")
 		(attr smd)
 		(fp_line
@@
 			)
 		)
+		(property ki_fp_filters "C_*")
+		(sheetname "Root")
+		(sheetfile "ScottoModules.kicad_sch")
 		(attr smd)
 		(fp_line
@@
 			)
 		)
+		(property ki_fp_filters "USB*C*Receptacle*")
+		(sheetname "Root")
+		(sheetfile "ScottoModules.kicad_sch")
 		(attr smd)
 		(fp_line
@@
 			)
 		)
+		(property "JlcRotOffset" "-90"
+			(at 0 0 90)
+			(unlocked yes)
+			(layer "B.Fab")
+			(hide yes)
+			(effects
+				(font
+					(size 1 1)
+					(thickness 0.15)
+				)
+				(justify mirror)
+			)
+		)
 		(attr smd)
 		(fp_line
@@
 			)
 		)
+		(property ki_fp_filters "C_*")
+		(sheetname "Root")
+		(sheetfile "ScottoModules.kicad_sch")
 		(attr smd)
 		(fp_line
@@
 			)
 		)
+		(sheetname "Root")
+		(sheetfile "ScottoModules.kicad_sch")
 		(attr smd)
 		(fp_line
@@
 			)
 		)
+		(property "JlcRotOffset" "-90"
+			(at 0 0 90)
+			(unlocked yes)
+			(layer "B.Fab")
+			(hide yes)
+			(effects
+				(font
+					(size 1 1)
+					(thickness 0.15)
+				)
+				(justify mirror)
+			)
+		)
+		(property ki_fp_filters "LQFP*7x7mm*P0.5mm*")
+		(sheetname "Root")
+		(sheetfile "ScottoModules.kicad_sch")
 		(attr smd)
+		(fp_circle
+			(center -3.75 3.75)
+			(end -3.625 3.75)
+			(stroke
+				(width 0.1)
+				(type solid)
+			)
+			(fill solid)
+			(layer "B.SilkS")
+		)
 		(fp_line
 			(start 3.15 -5.15)
@@
 			)
 		)
+		(property ki_fp_filters "C_*")
+		(sheetname "Root")
+		(sheetfile "ScottoModules.kicad_sch")
 		(attr smd)
 		(fp_line
@@
 			)
 		)
+		(sheetname "Root")
+		(sheetfile "ScottoModules.kicad_sch")
 		(attr smd)
 		(fp_line
@@
 			(layers "B.Cu")
 			(roundrect_rratio 0.1)
+			(net 52 "Net-(S1-Pad1)")
 			(pinfunction "1")
 			(pintype "passive")
@@
 			(layers "*.Cu" "*.Mask")
 			(remove_unused_layers no)
+			(net 52 "Net-(S1-Pad1)")
 			(pinfunction "1")
 			(pintype "passive")
@@
 			(layers "*.Cu" "*.Mask")
 			(remove_unused_layers no)
+			(net 49 "Net-(D4-A)")
 			(pinfunction "2")
 			(pintype "passive")
@@
 			(layers "B.Cu")
 			(roundrect_rratio 0.1)
+			(net 49 "Net-(D4-A)")
 			(pinfunction "2")
 			(pintype "passive")
@@
 			)
 		)
+		(property ki_fp_filters "C_*")
+		(sheetname "Root")
+		(sheetfile "ScottoModules.kicad_sch")
 		(attr smd)
 		(fp_line
@@
 			)
 		)
+		(sheetname "Root")
+		(sheetfile "ScottoModules.kicad_sch")
 		(attr smd)
 		(fp_line
@@
 			)
 		)
+		(property ki_fp_filters "C_*")
+		(sheetname "Root")
+		(sheetfile "ScottoModules.kicad_sch")
 		(attr smd)
 		(fp_line
@@
 			)
 		)
+		(property ki_fp_filters "R_*")
+		(sheetname "Root")
+		(sheetfile "ScottoModules.kicad_sch")
 		(attr smd)
 		(fp_line
@@
 			)
 		)
+		(sheetname "Root")
+		(sheetfile "ScottoModules.kicad_sch")
 		(attr smd)
 		(fp_line
@@
 			(layers "B.Cu")
 			(roundrect_rratio 0.1)
+			(net 54 "Net-(S3-Pad1)")
 			(pinfunction "1")
 			(pintype "passive")
@@
 			(layers "*.Cu" "*.Mask")
 			(remove_unused_layers no)
+			(net 54 "Net-(S3-Pad1)")
 			(pinfunction "1")
 			(pintype "passive")
@@
 			(layers "*.Cu" "*.Mask")
 			(remove_unused_layers no)
+			(net 51 "Net-(D6-A)")
 			(pinfunction "2")
 			(pintype "passive")
@@
 			(layers "B.Cu")
 			(roundrect_rratio 0.1)
+			(net 51 "Net-(D6-A)")
 			(pinfunction "2")
 			(pintype "passive")
@@
 			)
 		)
-		(property "Value" "100nf"
+		(property "Value" "100nF"
 			(at 0.000001 -1.159999 90)
 			(layer "B.Fab")
@@
 			)
 		)
+		(property ki_fp_filters "C_*")
+		(sheetname "Root")
+		(sheetfile "ScottoModules.kicad_sch")
 		(attr smd)
 		(fp_line
@@
 			)
 		)
+		(sheetname "Root")
+		(sheetfile "ScottoModules.kicad_sch")
 		(attr smd)
 		(fp_line
@@
 			)
 		)
+		(property "JlcRotOffset" "180"
+			(at 0 0 90)
+			(unlocked yes)
+			(layer "B.Fab")
+			(hide yes)
+			(effects
+				(font
+					(size 1 1)
+					(thickness 0.15)
+				)
+				(justify mirror)
+			)
+		)
 		(attr smd)
 		(fp_line
@@
 			)
 		)
+		(property ki_fp_filters "R_*")
+		(sheetname "Root")
+		(sheetfile "ScottoModules.kicad_sch")
 		(attr smd)
 		(fp_line
@@
 			)
 		)
+		(sheetname "Root")
+		(sheetfile "ScottoModules.kicad_sch")
 		(attr smd)
 		(fp_line
@@
 			)
 		)
+		(property ki_fp_filters "*Fuse*")
+		(sheetname "Root")
+		(sheetfile "ScottoModules.kicad_sch")
 		(attr smd)
 		(fp_line
@@
 			)
 		)
+		(sheetname "Root")
+		(sheetfile "ScottoModules.kicad_sch")
 		(attr smd)
 		(fp_line
@@
 			)
 		)
+		(sheetname "Root")
+		(sheetfile "ScottoModules.kicad_sch")
 		(attr smd)
 		(fp_line
@@
 			)
 		)
+		(sheetname "Root")
+		(sheetfile "ScottoModules.kicad_sch")
 		(attr smd)
 		(fp_line
@@
 			(layers "B.Cu")
 			(roundrect_rratio 0.1)
+			(net 52 "Net-(S1-Pad1)")
 			(pinfunction "1")
 			(pintype "passive")
@@
 			(layers "*.Cu" "*.Mask")
 			(remove_unused_layers no)
+			(net 52 "Net-(S1-Pad1)")
 			(pinfunction "1")
 			(pintype "passive")
@@
 			(layers "*.Cu" "*.Mask")
 			(remove_unused_layers no)
+			(net 49 "Net-(D4-A)")
 			(pinfunction "2")
 			(pintype "passive")
@@
 			(layers "B.Cu")
 			(roundrect_rratio 0.1)
+			(net 49 "Net-(D4-A)")
 			(pinfunction "2")
 			(pintype "passive")
@@
 			)
 		)
+		(property ki_fp_filters "C_*")
+		(sheetname "Root")
+		(sheetfile "ScottoModules.kicad_sch")
 		(attr smd)
 		(fp_line
@@
 			)
 		)
+		(sheetname "Root")
+		(sheetfile "ScottoModules.kicad_sch")
 		(attr smd)
 		(fp_line
