File: Extras/ScottoModules/ScottoModules.kicad_sch (KiCad schematic)
At the start: 30 parts, among them J1 USB_C, SW1 SW_Push, U1 STM32F072CBT6, U3 XC6206, U4 USBLC6-2SC6

Commit message: Fix JLCPCB Rotation
Parts:
- U1, U4: JlcRotOffset (none) -> -90
- U3: JlcRotOffset (none) -> 180
Changed lines of the file:
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@@
 		)
 		(instances
-			(project "ScottoController"
+			(project "ScottoModules"
 				(path "/92054fa3-5ad0-458e-bd73-acbcf8d11243"
 					(reference "#PWR06")
@@
 			)
 		)
+		(property "JlcRotOffset" "-90"
+			(at 45.72 120.65 0)
+			(effects
+				(font
+					(size 1.27 1.27)
+				)
+				(hide yes)
+			)
+		)
 		(pin "34"
 		)
@@
 		)
 		(instances
-			(project "ScottoController"
+			(project "ScottoModules"
 				(path "/92054fa3-5ad0-458e-bd73-acbcf8d11243"
 					(reference "U1")
@@
 			)
 		)
+		(property "JlcRotOffset" "180"
+			(at 256.54 143.51 0)
+			(effects
+				(font
+					(size 1.27 1.27)
+				)
+				(hide yes)
+			)
+		)
 		(pin "1"
 		)
@@
 		)
 		(instances
-			(project "ScottoController"
+			(project "ScottoModules"
 				(path "/92054fa3-5ad0-458e-bd73-acbcf8d11243"
 					(reference "U3")
@@
 		)
 		(instances
-			(project "ScottoController"
+			(project "ScottoModules"
 				(path "/92054fa3-5ad0-458e-bd73-acbcf8d11243"
 					(reference "#PWR010")
@@
 		)
 		(instances
-			(project "ScottoController"
+			(project "ScottoModules"
 				(path "/92054fa3-5ad0-458e-bd73-acbcf8d11243"
 					(reference "#PWR02")
@@
 		)
 		(instances
-			(project "ScottoController"
+			(project "ScottoModules"
 				(path "/92054fa3-5ad0-458e-bd73-acbcf8d11243"
 					(reference "C6")
@@
 		)
 		(instances
-			(project "ScottoController"
+			(project "ScottoModules"
 				(path "/92054fa3-5ad0-458e-bd73-acbcf8d11243"
 					(reference "S4")
@@
 		)
 		(instances
-			(project "ScottoController"
+			(project "ScottoModules"
 				(path "/92054fa3-5ad0-458e-bd73-acbcf8d11243"
 					(reference "R1")
@@
 		)
 		(instances
-			(project "ScottoController"
+			(project "ScottoModules"
 				(path "/92054fa3-5ad0-458e-bd73-acbcf8d11243"
 					(reference "#PWR016")
@@
 			)
 		)
+		(property "JlcRotOffset" "-90"
+			(at 215.9 135.89 0)
+			(effects
+				(font
+					(size 1.27 1.27)
+				)
+				(hide yes)
+			)
+		)
 		(pin "6"
 		)
@@
 		)
 		(instances
-			(project "ScottoController"
+			(project "ScottoModules"
 				(path "/92054fa3-5ad0-458e-bd73-acbcf8d11243"
 					(reference "U4")
@@
 		)
 		(instances
-			(project "ScottoController"
+			(project "ScottoModules"
 				(path "/92054fa3-5ad0-458e-bd73-acbcf8d11243"
 					(reference "#PWR04")
@@
 		)
 		(instances
-			(project "ScottoController"
+			(project "ScottoModules"
 				(path "/92054fa3-5ad0-458e-bd73-acbcf8d11243"
 					(reference "C8")
@@
 		)
 		(instances
-			(project "ScottoController"
+			(project "ScottoModules"
 				(path "/92054fa3-5ad0-458e-bd73-acbcf8d11243"
 					(reference "#PWR08")
@@
 		)
 		(instances
-			(project "ScottoController"
+			(project "ScottoModules"
 				(path "/92054fa3-5ad0-458e-bd73-acbcf8d11243"
 					(reference "#PWR07")
@@
 		)
 		(instances
-			(project "ScottoController"
+			(project "ScottoModules"
 				(path "/92054fa3-5ad0-458e-bd73-acbcf8d11243"
 					(reference "S2")
@@
 		)
 		(instances
-			(project "ScottoController"
+			(project "ScottoModules"
 				(path "/92054fa3-5ad0-458e-bd73-acbcf8d11243"
 					(reference "D2")
@@
 		)
 		(instances
-			(project "ScottoController"
+			(project "ScottoModules"
 				(path "/92054fa3-5ad0-458e-bd73-acbcf8d11243"
 					(reference "#PWR015")
@@
 		)
 		(instances
-			(project "ScottoController"
+			(project "ScottoModules"
 				(path "/92054fa3-5ad0-458e-bd73-acbcf8d11243"
 					(reference "D1")
@@
 		)
 		(instances
-			(project "ScottoController"
+			(project "ScottoModules"
 				(path "/92054fa3-5ad0-458e-bd73-acbcf8d11243"
 					(reference "C4")
@@
 		)
 		(instances
-			(project "ScottoController"
+			(project "ScottoModules"
 				(path "/92054fa3-5ad0-458e-bd73-acbcf8d11243"
 					(reference "S5")
@@
 		)
 		(instances
-			(project "ScottoController"
+			(project "ScottoModules"
 				(path "/92054fa3-5ad0-458e-bd73-acbcf8d11243"
 					(reference "C2")
@@
 		)
 		(instances
-			(project "ScottoController"
+			(project "ScottoModules"
 				(path "/92054fa3-5ad0-458e-bd73-acbcf8d11243"
 					(reference "#PWR03")
@@
 		)
 		(instances
-			(project "ScottoController"
+			(project "ScottoModules"
 				(path "/92054fa3-5ad0-458e-bd73-acbcf8d11243"
 					(reference "D5")
@@
 		)
 		(instances
-			(project "ScottoController"
+			(project "ScottoModules"
 				(path "/92054fa3-5ad0-458e-bd73-acbcf8d11243"
 					(reference "D4")
@@
 		)
 		(instances
-			(project "ScottoController"
+			(project "ScottoModules"
 				(path "/92054fa3-5ad0-458e-bd73-acbcf8d11243"
 					(reference "#PWR012")
@@
 		)
 		(instances
-			(project "ScottoController"
+			(project "ScottoModules"
 				(path "/92054fa3-5ad0-458e-bd73-acbcf8d11243"
 					(reference "C7")
@@
 		)
 		(instances
-			(project "ScottoController"
+			(project "ScottoModules"
 				(path "/92054fa3-5ad0-458e-bd73-acbcf8d11243"
 					(reference "D3")
@@
 		)
 		(instances
-			(project "ScottoController"
+			(project "ScottoModules"
 				(path "/92054fa3-5ad0-458e-bd73-acbcf8d11243"
 					(reference "#PWR01")
@@
 		)
 		(instances
-			(project "ScottoController"
+			(project "ScottoModules"
 				(path "/92054fa3-5ad0-458e-bd73-acbcf8d11243"
 					(reference "R3")
@@
 		)
 		(instances
-			(project "ScottoController"
+			(project "ScottoModules"
 				(path "/92054fa3-5ad0-458e-bd73-acbcf8d11243"
 					(reference "#PWR014")
@@
 		)
 		(instances
-			(project "ScottoController"
+			(project "ScottoModules"
 				(path "/92054fa3-5ad0-458e-bd73-acbcf8d11243"
 					(reference "#PWR013")
@@
 		)
 		(instances
-			(project "ScottoController"
+			(project "ScottoModules"
 				(path "/92054fa3-5ad0-458e-bd73-acbcf8d11243"
 					(reference "D6")
@@
 		)
 		(instances
-			(project "ScottoController"
+			(project "ScottoModules"
 				(path "/92054fa3-5ad0-458e-bd73-acbcf8d11243"
 					(reference "R2")
@@
 		)
 		(instances
-			(project "ScottoController"
+			(project "ScottoModules"
 				(path "/92054fa3-5ad0-458e-bd73-acbcf8d11243"
 					(reference "C3")
@@
 		)
 		(instances
-			(project "ScottoController"
+			(project "ScottoModules"
 				(path "/92054fa3-5ad0-458e-bd73-acbcf8d11243"
 					(reference "F1")
@@
 		)
 		(instances
-			(project "ScottoController"
+			(project "ScottoModules"
 				(path "/92054fa3-5ad0-458e-bd73-acbcf8d11243"
 					(reference "S6")
@@
 		)
 		(instances
-			(project "ScottoController"
+			(project "ScottoModules"
 				(path "/92054fa3-5ad0-458e-bd73-acbcf8d11243"
 					(reference "S1")
@@
 		)
 		(instances
-			(project "ScottoController"
+			(project "ScottoModules"
 				(path "/92054fa3-5ad0-458e-bd73-acbcf8d11243"
 					(reference "#PWR09")
@@
 		)
 		(instances
-			(project "ScottoController"
+			(project "ScottoModules"
 				(path "/92054fa3-5ad0-458e-bd73-acbcf8d11243"
 					(reference "S3")
@@
 		)
 		(instances
-			(project "ScottoController"
+			(project "ScottoModules"
 				(path "/92054fa3-5ad0-458e-bd73-acbcf8d11243"
 					(reference "J1")
@@
 		)
 		(instances
-			(project "ScottoController"
+			(project "ScottoModules"
 				(path "/92054fa3-5ad0-458e-bd73-acbcf8d11243"
 					(reference "C1")
@@
 		)
 		(instances
-			(project "ScottoController"
+			(project "ScottoModules"
 				(path "/92054fa3-5ad0-458e-bd73-acbcf8d11243"
 					(reference "#PWR05")
@@
 		)
 		(instances
-			(project "ScottoController"
+			(project "ScottoModules"
 				(path "/92054fa3-5ad0-458e-bd73-acbcf8d11243"
 					(reference "SW1")
@@
 		)
 		(instances
-			(project "ScottoController"
+			(project "ScottoModules"
 				(path "/92054fa3-5ad0-458e-bd73-acbcf8d11243"
 					(reference "C9")
@@
 		)
 		(instances
-			(project "ScottoController"
+			(project "ScottoModules"
 				(path "/92054fa3-5ad0-458e-bd73-acbcf8d11243"
 					(reference "C5")
@@
 		)
 		(instances
-			(project "ScottoController"
+			(project "ScottoModules"
 				(path "/92054fa3-5ad0-458e-bd73-acbcf8d11243"
 					(reference "#PWR011")
