File: Extras/ScottoModules/STM32F072CBT6/ScottoModules.kicad_pcb (KiCad board)
At the start: 4 copper layers, 38.1 x 57.2 mm, 26 parts, among them J1 USB_C, SW1 SW_Push, U1 STM32F072CBT6, U3 XC6206, U4 USBLC6-2SC6

Commit message: Regroup
Routing:
- net /BOOT0: track 22.6 -> 34.8 mm
- net /MCU_D-: track 7.85 -> 18.6 mm
- net /MCU_D+: track 7.85 -> 18.6 mm
- net +3.3V: track 62.0 -> 71.5 mm
Changed lines of the file:
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@@
+	)
+	(segment
+		(start 155.804945 114.612005)
+		(end 155.804945 105.949507)
+		(width 0.3)
+		(layer "F.Cu")
+		(net 2)
 	)
 	(segment
@@
 	)
 	(segment
-		(start 155.804945 114.612005)
-		(end 155.804945 105.949507)
+		(start 153.646196 95.589502)
+		(end 153.646196 105.030753)
 		(width 0.3)
 		(layer "F.Cu")
@@
 	)
 	(arc
+		(start 153.646196 105.030753)
+		(mid 153.915293 105.68041)
+		(end 154.56495 105.949507)
+		(width 0.3)
+		(layer "F.Cu")
+		(net 2)
+	)
+	(arc
 		(start 153.622445 116.794507)
 		(mid 155.165706 116.155268)
@@
 		(net 2)
 	)
-	(arc
-		(start 153.646196 105.030753)
-		(mid 153.915293 105.68041)
-		(end 154.56495 105.949507)
-		(width 0.3)
-		(layer "F.Cu")
-		(net 2)
-	)
 	(segment
 		(start 152.912445 106.989505)
@@
 	)
 	(segment
+		(start 150.912445 96.235031)
+		(end 150.912445 106.989505)
+		(width 0.2)
+		(layer "B.Cu")
+		(net 23)
+	)
+	(segment
 		(start 150.912447 90.680563)
 		(end 150.912447 96.235029)
@@
 		(start 150.912447 106.989503)
 		(end 150.912445 106.989505)
+		(width 0.2)
+		(layer "B.Cu")
+		(net 23)
+	)
+	(segment
+		(start 150.912447 96.235029)
+		(end 150.912445 96.235031)
 		(width 0.2)
 		(layer "B.Cu")
@@
 	)
 	(segment
+		(start 151.412445 96.235031)
+		(end 151.412445 106.989505)
+		(width 0.2)
+		(layer "B.Cu")
+		(net 24)
+	)
+	(segment
 		(start 151.412447 90.680553)
 		(end 151.412447 96.235029)
+		(width 0.2)
+		(layer "B.Cu")
+		(net 24)
+	)
+	(segment
+		(start 151.412447 96.235029)
+		(end 151.412445 96.235031)
 		(width 0.2)
 		(layer "B.Cu")
@@
 		(layer "B.Cu")
 		(net 25)
+	)
+	(segment
+		(start 149.912445 96.239502)
+		(end 149.912445 108.489505)
+		(width 0.2)
+		(layer "F.Cu")
+		(net 26)
 	)
 	(via
@@
 			"889fd9f7-8632-4145-94b1-e8dfb995efd2" "89d405ed-2f5c-44c8-8711-8e3c12c85794"
 			"8ac0805e-693d-42f8-83eb-69217bb2bcd5" "963c4cf8-b45e-4feb-94ad-1bdae0c02658"
-			"98b004fa-ecf0-4b5f-8622-3f85478b17a0" "99ce805b-7fa7-4d11-afc8-944c7437d551"
-			"9a56ebde-bfc3-4511-b692-6430f33ed308" "9b8d5076-778b-4a70-99f0-d5e6d5716dd4"
-			"9f9e6d95-7f27-40d6-bbc2-0efe381c19bd" "a02fac82-1e78-4b3f-a629-10eb105dcf31"
+			"99ce805b-7fa7-4d11-afc8-944c7437d551" "9a56ebde-bfc3-4511-b692-6430f33ed308"
+			"9b8d5076-778b-4a70-99f0-d5e6d5716dd4" "a02fac82-1e78-4b3f-a629-10eb105dcf31"
 			"a3f4f0e7-65cc-4128-bebc-e7ce49d8d615" "aa6ccd1b-89ae-4b45-a839-1ac306b56670"
 			"ab83ab6b-6ef4-4512-8017-cc87d65aab55" "ae219cc8-5654-4e36-9d64-7c2c31208421"
