File: Extras/ScottoModules/STM32F072CBT6/ScottoModules.kicad_sch (KiCad schematic)
At the start: 18 parts, among them J1 USB_C, SW1 SW_Push, U1 STM32F072CBT6, U3 XC6206, U4 USBLC6-2SC6

Commit message: Update to better V2
Parts:
- removed C1, C2, C3, C4, C5: 100nF, ScottoKeebs_Components:Capacitor_0402, symbol Device:C_Small
- removed C6: 10uF, ScottoKeebs_Components:Capacitor_0603, symbol Device:C_Small
- added C10, C11, C13, C16: 100nF, ScottoKeebs_Components:Capacitor_0402, symbol Device:C_Small
- added C12, C17: 4.7uF, ScottoKeebs_Components:Capacitor_0402, symbol Device:C_Small
- added C14: 10nF, ScottoKeebs_Components:Capacitor_0402, symbol Device:C_Small
- added C15: 1uF, ScottoKeebs_Components:Capacitor_0402, symbol Device:C_Small
Connections:
- net +3.3V: now also C10.2, C11.2, C12.2, C13.2, C14.2, C15.2, C16.2, C17.2
- net +5V: no longer U4.5 (VBUS)
- net GND: now also C10.1, C11.1, C12.1, C13.1, C14.1, C15.1, C16.1, C17.1
- net VBUS: now also U4.5 (VBUS)
- net NRST: now reaches C7.1, U1.7 (NRST)
- net D+ renamed USB_D+
- net USB_D+: no longer U1.33 (PA12), U4.1 (I/O1)
- net D- renamed USB_D-
- net USB_D-: no longer U1.32 (PA11), U4.3 (I/O2)
- new net MCU_D+: U1.33 (PA12), U4.1 (I/O1)
- new net MCU_D-: U1.32 (PA11), U4.3 (I/O2)
Other:
- note added: "Power Flags"
- moved on the sheet: C7, U1

Commit message: Should be final
Other:
- note added: "Matrix"
- note added: "Mounting Holes"
- note added: "Other"
- moved on the sheet: C10, C11, C12, C13, C14, C15, C16, C17, C8, C9, F1, J1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
